Commit message: modified maze to give more room to the robot to move

File: turtlebot3_simulations/turtlebot3_gazebo/urdf/turtlebot3_waffle.urdf (robot description, URDF)
Before this commit: robot turtlebot3_waffle, 14 links, 13 joints
Links:
- link logical_camera_link: geometry visual mesh filename=package://turtlebot3_gazebo/models/advanced_logical_camera/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 scale=0.001 0.001 0.001
